File: board/flash.sch (KiCad schematic (older format))
At the start: 4 parts, among them U1501 W25Q64JVSSIM

Commit message: Most footprints associated
Parts:
- C1501: footprint (none) -> Capacitor_SMD:C_0603_1608Metric
- R1501, R1502: footprint (none) -> Resistor_SMD:R_0603_1608Metric
- U1501: footprint (none) -> Package_SO:SOIJ-8_5.3x5.3mm_P1.27mm
Changed lines of the file:
@@
 F 0 "U1501" H 3325 4640 50  0000 C CNN
 F 1 "W25Q64JVSSIM" H 3325 4549 50  0000 C CNN
-F 2 "" H 3050 4375 50  0001 C CNN
+F 2 "Package_SO:SOIJ-8_5.3x5.3mm_P1.27mm" H 3050 4375 50  0001 C CNN
 F 3 "" H 3050 4375 50  0001 C CNN
 	1    3325 4225
@@
 F 0 "R1502" V 2800 4125 50  0000 C CNN
 F 1 "4K7" V 2700 4275 50  0000 C CNN
-F 2 "" V 2630 4275 50  0001 C CNN
+F 2 "Resistor_SMD:R_0603_1608Metric" V 2630 4275 50  0001 C CNN
 F 3 "~" H 2700 4275 50  0001 C CNN
 	1    2700 4275
@@
 F 0 "R1501" V 3875 4200 50  0000 C CNN
 F 1 "4K7" V 3950 4175 50  0000 C CNN
-F 2 "" V 3880 4175 50  0001 C CNN
+F 2 "Resistor_SMD:R_0603_1608Metric" V 3880 4175 50  0001 C CNN
 F 3 "~" H 3950 4175 50  0001 C CNN
 	1    3950 4175
@@
 F 0 "C1501" H 4615 4271 50  0000 L CNN
 F 1 "1u" H 4615 4180 50  0000 L CNN
-F 2 "" H 4538 4075 50  0001 C CNN
+F 2 "Capacitor_SMD:C_0603_1608Metric" H 4538 4075 50  0001 C CNN
 F 3 "~" H 4500 4225 50  0001 C CNN
 	1    4500 4225
