File: board/sub_gpio.sch (KiCad schematic (older format))
At the start: 22 parts, among them J401 Conn_01x09, U401 74LVC4245A

Commit message: More footprints done. Went with simpler test-pads.
Parts:
- J401: footprint (none) -> Connector_PinHeader_2.54mm:PinHeader_1x09_P2.54mm_Vertical
Changed lines of the file:
@@
 $Descr A4 11693 8268
 encoding utf-8
-Sheet 4 15
+Sheet 4 14
 Title ""
 Date ""
@@
 F 0 "J401" H 2145 3517 50  0000 C CNN
 F 1 "Conn_01x09" H 2145 3426 50  0000 C CNN
-F 2 "" H 2225 2900 50  0001 C CNN
+F 2 "Connector_PinHeader_2.54mm:PinHeader_1x09_P2.54mm_Vertical" H 2225 2900 50  0001 C CNN
 F 3 "~" H 2225 2900 50  0001 C CNN
 	1    2225 2900

Commit message: Most footprints associated
Parts:
- C401, C402: footprint (none) -> Capacitor_SMD:C_0603_1608Metric
- D403, D404, D405, D406, D407, D408, D409, D410: footprint (none) -> LED_SMD:LED_0805_2012Metric
- R401, R402, R403, R404, R405, R406, R407, R408: footprint (none) -> Resistor_SMD:R_0603_1608Metric
Changed lines of the file:
@@
 F 0 "C401" H 6915 2896 50  0000 L CNN
 F 1 "1u" H 6915 2805 50  0000 L CNN
-F 2 "" H 6838 2700 50  0001 C CNN
+F 2 "Capacitor_SMD:C_0603_1608Metric" H 6838 2700 50  0001 C CNN
 F 3 "~" H 6800 2850 50  0001 C CNN
 	1    6800 2850
@@
 F 0 "D403" H 4150 3550 50  0000 R CNN
 F 1 "LED_Small" V 3855 3432 50  0001 R CNN
-F 2 "" V 3900 3500 50  0001 C CNN
+F 2 "LED_SMD:LED_0805_2012Metric" V 3900 3500 50  0001 C CNN
 F 3 "~" V 3900 3500 50  0001 C CNN
 	1    3900 3500
@@
 F 0 "D410" H 4850 3550 50  0000 R CNN
 F 1 "LED_Small" V 4555 3432 50  0001 R CNN
-F 2 "" V 4600 3500 50  0001 C CNN
+F 2 "LED_SMD:LED_0805_2012Metric" V 4600 3500 50  0001 C CNN
 F 3 "~" V 4600 3500 50  0001 C CNN
 	1    4600 3500
@@
 F 0 "D409" H 4750 3550 50  0000 R CNN
 F 1 "LED_Small" V 4455 3432 50  0001 R CNN
-F 2 "" V 4500 3500 50  0001 C CNN
+F 2 "LED_SMD:LED_0805_2012Metric" V 4500 3500 50  0001 C CNN
 F 3 "~" V 4500 3500 50  0001 C CNN
 	1    4500 3500
@@
 F 0 "D408" H 4650 3550 50  0000 R CNN
 F 1 "LED_Small" V 4355 3432 50  0001 R CNN
-F 2 "" V 4400 3500 50  0001 C CNN
+F 2 "LED_SMD:LED_0805_2012Metric" V 4400 3500 50  0001 C CNN
 F 3 "~" V 4400 3500 50  0001 C CNN
 	1    4400 3500
@@
 F 0 "D407" H 4550 3550 50  0000 R CNN
 F 1 "LED_Small" V 4255 3432 50  0001 R CNN
-F 2 "" V 4300 3500 50  0001 C CNN
+F 2 "LED_SMD:LED_0805_2012Metric" V 4300 3500 50  0001 C CNN
 F 3 "~" V 4300 3500 50  0001 C CNN
 	1    4300 3500
@@
 F 0 "D406" H 4450 3550 50  0000 R CNN
 F 1 "LED_Small" V 4155 3432 50  0001 R CNN
-F 2 "" V 4200 3500 50  0001 C CNN
+F 2 "LED_SMD:LED_0805_2012Metric" V 4200 3500 50  0001 C CNN
 F 3 "~" V 4200 3500 50  0001 C CNN
 	1    4200 3500
@@
 F 0 "D405" H 4350 3550 50  0000 R CNN
 F 1 "LED_Small" V 4055 3432 50  0001 R CNN
-F 2 "" V 4100 3500 50  0001 C CNN
+F 2 "LED_SMD:LED_0805_2012Metric" V 4100 3500 50  0001 C CNN
 F 3 "~" V 4100 3500 50  0001 C CNN
 	1    4100 3500
@@
 F 0 "D404" H 4250 3550 50  0000 R CNN
 F 1 "LED_Small" V 3955 3432 50  0001 R CNN
-F 2 "" V 4000 3500 50  0001 C CNN
+F 2 "LED_SMD:LED_0805_2012Metric" V 4000 3500 50  0001 C CNN
 F 3 "~" V 4000 3500 50  0001 C CNN
 	1    4000 3500
@@
 F 0 "R401" V 3850 3400 50  0000 L CNN
 F 1 "390" V 3900 3675 50  0000 L CNN
-F 2 "" V 3830 3750 50  0001 C CNN
+F 2 "Resistor_SMD:R_0603_1608Metric" V 3830 3750 50  0001 C CNN
 F 3 "~" H 3900 3750 50  0001 C CNN
 	1    3900 3750
@@
 F 0 "R402" V 3950 3400 50  0000 L CNN
 F 1 "390" V 4000 3675 50  0000 L CNN
-F 2 "" V 3930 3750 50  0001 C CNN
+F 2 "Resistor_SMD:R_0603_1608Metric" V 3930 3750 50  0001 C CNN
 F 3 "~" H 4000 3750 50  0001 C CNN
 	1    4000 3750
@@
 F 0 "R403" V 4050 3400 50  0000 L CNN
 F 1 "390" V 4100 3675 50  0000 L CNN
-F 2 "" V 4030 3750 50  0001 C CNN
+F 2 "Resistor_SMD:R_0603_1608Metric" V 4030 3750 50  0001 C CNN
 F 3 "~" H 4100 3750 50  0001 C CNN
 	1    4100 3750
@@
 F 0 "R404" V 4150 3400 50  0000 L CNN
 F 1 "390" V 4200 3675 50  0000 L CNN
-F 2 "" V 4130 3750 50  0001 C CNN
+F 2 "Resistor_SMD:R_0603_1608Metric" V 4130 3750 50  0001 C CNN
 F 3 "~" H 4200 3750 50  0001 C CNN
 	1    4200 3750
@@
 F 0 "R405" V 4250 3400 50  0000 L CNN
 F 1 "390" V 4300 3675 50  0000 L CNN
-F 2 "" V 4230 3750 50  0001 C CNN
+F 2 "Resistor_SMD:R_0603_1608Metric" V 4230 3750 50  0001 C CNN
 F 3 "~" H 4300 3750 50  0001 C CNN
 	1    4300 3750
@@
 F 0 "R406" V 4350 3400 50  0000 L CNN
 F 1 "390" V 4400 3675 50  0000 L CNN
-F 2 "" V 4330 3750 50  0001 C CNN
+F 2 "Resistor_SMD:R_0603_1608Metric" V 4330 3750 50  0001 C CNN
 F 3 "~" H 4400 3750 50  0001 C CNN
 	1    4400 3750
@@
 F 0 "R407" V 4450 3400 50  0000 L CNN
 F 1 "390" V 4500 3675 50  0000 L CNN
-F 2 "" V 4430 3750 50  0001 C CNN
+F 2 "Resistor_SMD:R_0603_1608Metric" V 4430 3750 50  0001 C CNN
 F 3 "~" H 4500 3750 50  0001 C CNN
 	1    4500 3750
@@
 F 0 "R408" V 4550 3400 50  0000 L CNN
 F 1 "390" V 4600 3675 50  0000 L CNN
-F 2 "" V 4530 3750 50  0001 C CNN
+F 2 "Resistor_SMD:R_0603_1608Metric" V 4530 3750 50  0001 C CNN
 F 3 "~" H 4600 3750 50  0001 C CNN
 	1    4600 3750
@@
 F 0 "C402" H 7415 2896 50  0000 L CNN
 F 1 "1u" H 7415 2805 50  0000 L CNN
-F 2 "" H 7338 2700 50  0001 C CNN
+F 2 "Capacitor_SMD:C_0603_1608Metric" H 7338 2700 50  0001 C CNN
 F 3 "~" H 7300 2850 50  0001 C CNN
 	1    7300 2850
