File: board/sub_ram.sch (KiCad schematic (older format))
At the start: 2 parts, among them U1101 AS6C8008

Commit message: Most footprints associated
Parts:
- C1101: footprint (none) -> Capacitor_SMD:C_0603_1608Metric
Changed lines of the file:
@@
 F 0 "C1101" H 6865 3346 50  0000 L CNN
 F 1 "1u" H 6865 3255 50  0000 L CNN
-F 2 "" H 6788 3150 50  0001 C CNN
+F 2 "Capacitor_SMD:C_0603_1608Metric" H 6788 3150 50  0001 C CNN
 F 3 "~" H 6750 3300 50  0001 C CNN
 	1    6750 3300

Commit message: Almost all footprints done
Parts:
- U1101: footprint (none) -> quokka:AS6C8008-SOIC-44
Changed lines of the file:
@@
 F 0 "U1101" H 5075 3825 50  0000 C CNN
 F 1 "AS6C8008" H 5625 3825 50  0000 C CNN
-F 2 "" H 5000 3125 50  0001 C CNN
+F 2 "quokka:AS6C8008-SOIC-44" H 5000 3125 50  0001 C CNN
 F 3 "https://www.alliancememory.com/wp-content/uploads/pdf/AS6C8008.pdf" H 5000 3125 50  0001 C CNN
 	1    5400 2675
