File: board/sub_power.sch (KiCad schematic (older format))
At the start: 70 parts, among them J201 Barrel_Jack, Q201 Q_PMOS_GSD, U201 TS3001x, U202 TS3001x, U203 LDL1117S25R, U204 LDL1117S12R, U205 XC3S200-TQ144

Commit message: Most footprints associated
Parts:
- C201, C206, C214, C215, C216, C217, C218, C219, C220, C221, C222, C223, C224, C225, C226, C227, C228, C229, C230, C231, C232, C233, C234, C235, C236, C237, C238, C239, C240, C241, C242, C243, C244, C245, C246, C247, C248, C249: footprint (none) -> Capacitor_SMD:C_0603_1608Metric
- C202, C203, C205, C210: footprint (none) -> Capacitor_SMD:C_1206_3216Metric
- C204: footprint (none) -> Capacitor_THT:CP_Radial_D6.3mm_P2.50mm
- C207, C208, C211, C212: footprint (none) -> Capacitor_SMD:C_0805_2012Metric
- C209, C213: footprint (none) -> Capacitor_THT:CP_Radial_D8.0mm_P3.50mm
- D201: footprint (none) -> Diode_SMD:D_SMA
- D202, D203: footprint (none) -> Diode_SMD:D_SOD-123F
- L201: value L_Coupled -> Power Choke
- L202, L203: footprint (none) -> Inductor_SMD:L_Taiyo-Yuden_NR-60xx

Commit message: All footprints done
Parts:
- L201: footprint (none) -> quokka:CM2021Y330R-10
Changed lines of the file:
@@
 F 0 "L201" H 2450 1162 50  0000 C CNN
 F 1 "Power Choke" H 2450 1162 50  0001 C CNN
-F 2 "" H 2450 975 50  0001 C CNN
+F 2 "quokka:CM2021Y330R-10" H 2450 975 50  0001 C CNN
 F 3 "~" H 2450 975 50  0001 C CNN
 	1    2450 975

Commit message: Power supply routed
Parts:
- TP201, TP202, TP203, TP204, TP205, TP206: footprint TestPoint:TestPoint_Plated_Hole_D2.0mm -> TestPoint:TestPoint_Pad_D1.5mm
Changed lines of the file:
@@
 F 0 "TP201" H 1258 874 50  0000 L CNN
 F 1 "Test_Point" H 1258 829 50  0001 L CNN
-F 2 "TestPoint:TestPoint_Plated_Hole_D2.0mm" H 1400 800 50  0001 C CNN
+F 2 "TestPoint:TestPoint_Pad_D1.5mm" H 1400 800 50  0001 C CNN
 F 3 "~" H 1400 800 50  0001 C CNN
 	1    1200 800
@@
 F 0 "TP202" V 3800 900 50  0000 L CNN
 F 1 "Test_Point" H 3783 904 50  0001 L CNN
-F 2 "TestPoint:TestPoint_Plated_Hole_D2.0mm" H 3925 875 50  0001 C CNN
+F 2 "TestPoint:TestPoint_Pad_D1.5mm" H 3925 875 50  0001 C CNN
 F 3 "~" H 3925 875 50  0001 C CNN
 	1    3725 875
@@
 F 0 "TP203" H 6250 1300 50  0000 L CNN
 F 1 "Test_Point" H 6433 1104 50  0001 L CNN
-F 2 "TestPoint:TestPoint_Plated_Hole_D2.0mm" H 6575 1075 50  0001 C CNN
+F 2 "TestPoint:TestPoint_Pad_D1.5mm" H 6575 1075 50  0001 C CNN
 F 3 "~" H 6575 1075 50  0001 C CNN
 	1    6375 1075
@@
 F 0 "TP204" H 9750 1500 50  0000 L CNN
 F 1 "Test_Point" H 9933 1304 50  0001 L CNN
-F 2 "TestPoint:TestPoint_Plated_Hole_D2.0mm" H 10075 1275 50  0001 C CNN
+F 2 "TestPoint:TestPoint_Pad_D1.5mm" H 10075 1275 50  0001 C CNN
 F 3 "~" H 10075 1275 50  0001 C CNN
 	1    9875 1275
@@
 F 0 "TP205" H 2575 2825 50  0000 L CNN
 F 1 "Test_Point" H 2758 2629 50  0001 L CNN
-F 2 "TestPoint:TestPoint_Plated_Hole_D2.0mm" H 2900 2600 50  0001 C CNN
+F 2 "TestPoint:TestPoint_Pad_D1.5mm" H 2900 2600 50  0001 C CNN
 F 3 "~" H 2900 2600 50  0001 C CNN
 	1    2700 2600
@@
 F 0 "TP206" V 3675 2775 50  0000 L CNN
 F 1 "Test_Point" H 3733 2629 50  0001 L CNN
-F 2 "TestPoint:TestPoint_Plated_Hole_D2.0mm" H 3875 2600 50  0001 C CNN
+F 2 "TestPoint:TestPoint_Pad_D1.5mm" H 3875 2600 50  0001 C CNN
 F 3 "~" H 3875 2600 50  0001 C CNN
 	1    3675 2600
