File: board/quokka.kicad_pcb (KiCad board)
At the start: 4 copper layers, 341 parts, among them J1301 FPGA JTAG, J201 Barrel_Jack, J301 ARM SWD, J302 Conn_01x02, J303 Conn_01x09, J304 Conn_01x03, J305 USB_B, J401 Conn_01x09, Q1201 Q_NPN_BEC, Q1301 Q_NPN_BEC, Q1401 Q_NPN_BEC, Q1402 Q_NPN_BEC, Q1403 Q_NPN_BEC, Q201 Q_PMOS_GSD, Q601 Q_PMOS_GSD, Q602 Q_PMOS_GSD, Q603 Q_PMOS_GSD, Q604 Q_PMOS_GSD, Q605 Q_PMOS_GSD, Q606 Q_PMOS_GSD, Q607 Q_PMOS_GSD, Q608 Q_PMOS_GSD, Q701 Q_PMOS_GSD, Q702 Q_PMOS_GSD, Q703 Q_PMOS_GSD, Q704 Q_PMOS_GSD, Q705 Q_PMOS_GSD, Q706 Q_PMOS_GSD, Q707 Q_PMOS_GSD, Q708 Q_PMOS_GSD, Q801 Q_PMOS_GSD, Q802 Q_PMOS_GSD, Q803 Q_PMOS_GSD, Q804 Q_PMOS_GSD, Q805 Q_PMOS_GSD, Q806 Q_PMOS_GSD, Q807 Q_PMOS_GSD, SW901 SW_SPST, SW902 SW_SPST, SW903 SW_SPST, SW904 SW_SPST, SW905 SW_SPST, SW906 SW_SPST, SW907 SW_SPST, SW908 SW_SPST, SW909 SW_SPST, SW910 SW_SPST, SW911 SW_SPST, SW912 SW_SPST, SW913 SW_SPST, SW914 SW_SPST, SW915 SW_SPST, SW916 SW_SPST, SW917 SW_SPST, SW918 SW_SPST, SW919 SW_SPST, SW920 SW_SPST, SW921 SW_SPST, SW922 SW_SPST, SW923 SW_SPST, SW924 SW_SPST, SW925 SW_SPST, SW926 SW_SPST, SW927 SW_SPST, SW928 SW_SPST, SW929 SW_SPST, SW930 SW_SPST, U1001 DIN96, U1101 AS6C8008, U1201 74HCT245, U1202 6502, U1203 74HCT245, U1204 74HCT245, U1205 74HCT245, U1401 74LVC4245A, U1402 74LVC4245A, U1403 74LVC4245A, U1404 74LVC4245A, U1405 74LVC4245A, U1406 74LVC4245A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

Commit message: more progress on board
Parts:
- moved C701 284.9 mm to (5.15, 120.3)
- moved C702 284.9 mm to (5.15, 114.9)
- moved R705 284.9 mm to (15.5, 100.0)
- moved R706 284.9 mm to (10.2, 113.2)
- moved R707 284.9 mm to (-5.69, 128.1)
- moved R708 284.9 mm to (-10.2, 133.5)
- moved C703 284.9 mm to (15.4, 110.7)
- moved R701 284.9 mm to (-10.1, 128.1)
- moved R702 284.9 mm to (-0.03, 121.1)
- moved R703 284.9 mm to (15.4, 105.3)
- moved R704 284.9 mm to (-0.03, 126.4)
- moved U602 250.7 mm to (59.7, 77.5)
- moved U802 249.0 mm to (59.7, 43.2)
- moved U603 239.8 mm to (59.7, 66.0)
- moved R722 234.2 mm to (68.6, 105.4)
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Connections:
- U601 pad 11: Net-(Q602-Pad1) -> Net-(Q606-Pad1)
- U601 pad 12: Net-(Q606-Pad1) -> Net-(Q602-Pad1)
- U601 pad 13: Net-(Q601-Pad1) -> Net-(Q605-Pad1)
- U601 pad 14: Net-(Q605-Pad1) -> Net-(Q601-Pad1)
- U601 pad 3: Net-(Q604-Pad1) -> Net-(Q607-Pad1)
- U601 pad 4: Net-(Q608-Pad1) -> Net-(Q603-Pad1)
- U601 pad 5: Net-(Q603-Pad1) -> Net-(Q608-Pad1)
- U601 pad 6: Net-(Q607-Pad1) -> Net-(Q604-Pad1)
- U602 pad 11: Net-(R613-Pad1) -> Net-(R614-Pad1)
- U602 pad 12: Net-(R614-Pad1) -> Net-(R613-Pad1)
- U602 pad 13: Net-(R615-Pad1) -> Net-(R616-Pad1)
- U602 pad 14: Net-(R616-Pad1) -> Net-(R615-Pad1)
- U602 pad 3: Net-(R609-Pad1) -> Net-(R612-Pad1)
- U602 pad 4: Net-(R610-Pad1) -> Net-(R611-Pad1)
- U602 pad 5: Net-(R611-Pad1) -> Net-(R610-Pad1)
- U602 pad 6: Net-(R612-Pad1) -> Net-(R609-Pad1)
- U603 pad 11: Net-(R621-Pad1) -> Net-(R622-Pad1)
- U603 pad 12: Net-(R622-Pad1) -> Net-(R621-Pad1)
- U603 pad 13: Net-(R623-Pad1) -> Net-(U603-Pad13)
- U603 pad 14: Net-(U603-Pad14) -> Net-(R623-Pad1)
- U603 pad 3: Net-(R617-Pad1) -> Net-(R620-Pad1)
- U603 pad 4: Net-(R618-Pad1) -> Net-(R619-Pad1)
- U603 pad 5: Net-(R619-Pad1) -> Net-(R618-Pad1)
- U603 pad 6: Net-(R620-Pad1) -> Net-(R617-Pad1)
- U701 pad 11: Net-(Q702-Pad1) -> Net-(Q706-Pad1)
- U701 pad 12: Net-(Q706-Pad1) -> Net-(Q702-Pad1)
- U701 pad 13: Net-(Q701-Pad1) -> Net-(Q705-Pad1)
- U701 pad 14: Net-(Q705-Pad1) -> Net-(Q701-Pad1)
- U701 pad 3: Net-(Q704-Pad1) -> Net-(Q707-Pad1)
- U701 pad 4: Net-(Q708-Pad1) -> Net-(Q703-Pad1)
- U701 pad 5: Net-(Q703-Pad1) -> Net-(Q708-Pad1)
- U701 pad 6: Net-(Q707-Pad1) -> Net-(Q704-Pad1)
- U702 pad 11: Net-(R713-Pad1) -> Net-(R714-Pad1)
- U702 pad 12: Net-(R714-Pad1) -> Net-(R713-Pad1)
- U702 pad 13: Net-(R715-Pad1) -> Net-(R716-Pad1)
- U702 pad 14: Net-(R716-Pad1) -> Net-(R715-Pad1)
- U702 pad 3: Net-(R709-Pad1) -> Net-(R712-Pad1)
- U702 pad 4: Net-(R710-Pad1) -> Net-(R711-Pad1)
- U702 pad 5: Net-(R711-Pad1) -> Net-(R710-Pad1)
- U702 pad 6: Net-(R712-Pad1) -> Net-(R709-Pad1)
- U703 pad 11: Net-(R721-Pad1) -> Net-(R722-Pad1)
- U703 pad 12: Net-(R722-Pad1) -> Net-(R721-Pad1)
- U703 pad 13: Net-(R723-Pad1) -> Net-(U703-Pad13)
- U703 pad 14: Net-(U703-Pad14) -> Net-(R723-Pad1)
- U703 pad 3: Net-(R717-Pad1) -> Net-(R720-Pad1)
- U703 pad 4: Net-(R718-Pad1) -> Net-(R719-Pad1)
- U703 pad 5: Net-(R719-Pad1) -> Net-(R718-Pad1)
- U703 pad 6: Net-(R720-Pad1) -> Net-(R717-Pad1)
- U801 pad 11: Net-(Q802-Pad1) -> Net-(Q805-Pad1)
- U801 pad 12: Net-(Q805-Pad1) -> Net-(Q802-Pad1)
- U801 pad 13: Net-(Q801-Pad1) -> Net-(Q804-Pad1)
- U801 pad 14: Net-(Q804-Pad1) -> Net-(Q801-Pad1)
- U801 pad 3: Net-(Q807-Pad1) -> Net-(Q806-Pad1)
- U801 pad 4: Net-(Q807-Pad1) -> Net-(Q803-Pad1)
- U801 pad 5: Net-(Q803-Pad1) -> Net-(Q807-Pad1)
- U801 pad 6: Net-(Q806-Pad1) -> Net-(Q807-Pad1)
- U802 pad 11: Net-(R812-Pad1) -> Net-(R813-Pad1)
- U802 pad 12: Net-(R813-Pad1) -> Net-(R812-Pad1)
- U802 pad 13: Net-(R814-Pad1) -> Net-(R815-Pad1)
- U802 pad 14: Net-(R815-Pad1) -> Net-(R814-Pad1)
- U802 pad 3: Net-(R808-Pad1) -> Net-(R811-Pad1)
- U802 pad 4: Net-(R809-Pad1) -> Net-(R810-Pad1)
- U802 pad 5: Net-(R810-Pad1) -> Net-(R809-Pad1)
- U802 pad 6: Net-(R811-Pad1) -> Net-(R808-Pad1)
- U803 pad 11: Net-(R820-Pad1) -> Net-(R821-Pad1)
- U803 pad 12: Net-(R821-Pad1) -> Net-(R820-Pad1)
- U803 pad 13: Net-(R822-Pad1) -> Net-(R823-Pad1)
- U803 pad 14: Net-(R823-Pad1) -> Net-(R822-Pad1)
- U803 pad 3: Net-(R816-Pad1) -> Net-(R819-Pad1)
- U803 pad 4: Net-(R817-Pad1) -> Net-(R818-Pad1)
- U803 pad 5: Net-(R818-Pad1) -> Net-(R817-Pad1)
- U803 pad 6: Net-(R819-Pad1) -> Net-(R816-Pad1)

Commit message: Power supply routed
Parts:
- removed D814, D815, D816: LED_Small, LED_SMD:LED_0805_2012Metric
- removed R823: 160, Resistor_SMD:R_1206_3216Metric
- C1301, C218, C219, C220, C221, C222, C223, C224, C225, C226, C227, C228, C229, C230, C231, C232, C233, C234, C235, C236, C237, C238, C239, C240, C241, C242, C243, C244, C245, C246, C247, C248, C249, C301, C302, C303, C304, C305, C306, C402, C601, C602, C603, C701, C703, C801, C802, C803, Q601, Q602, Q603, Q604, Q605, Q606, Q607, Q608, Q701, Q702, Q703, Q704, Q705, Q706, Q708, Q801, Q802, Q803, Q804, Q805, Q806, Q807, R401, R402, R403, R404, R405, R406, R407, R408, R601, R602, R603, R604, R605, R606, R607, R608, R610, R612, R614, R616, R618, R620, R621, R623, R701, R702, R703, R704, R705, R706, R708, R710, R712, R714, R716, R718, R720, R721, R723, R801, R802, R803, R804, R805, R806, R807, R809, R811, R813, R815, R817, R818, R820: moved to B.Cu
- TP201, TP202, TP203, TP204, TP205, TP206: footprint TestPoint:TestPoint_Plated_Hole_D2.0mm -> TestPoint:TestPoint_Pad_D1.5mm
- moved U1204 421.9 mm to (201.1, 175.5), turned to 180 degrees
- moved C1204 421.8 mm to (196.1, 188.2), turned to 180 degrees
- moved U1203 420.5 mm to (201.1, 184.4), turned to 180 degrees
- moved U1201 418.1 mm to (201.1, 157.8), turned to 180 degrees
- moved C1205 412.6 mm to (196.1, 179.4), turned to 180 degrees
- moved U1202 411.8 mm to (171.7, 147.6)
- moved C1206 409.9 mm to (196.1, 170.5), turned to 180 degrees
- moved JP1201 409.6 mm to (198.6, 137.4), turned to 270 degrees
- moved R1203 408.6 mm to (199.9, 150.1)
- moved C1201 406.2 mm to (196.1, 161.6), turned to 180 degrees
- moved U1205 403.5 mm to (201.1, 166.7), turned to 180 degrees
- moved R1202 402.9 mm to (194.2, 157.8), turned to 180 degrees
- moved JP1202 401.8 mm to (198.6, 142.5), turned to 270 degrees
- moved Q1201 395.0 mm to (196.1, 148.9), turned to 180 degrees
- moved C1202 377.0 mm to (165.6, 164.1), turned to 90 degrees
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Connections:
- net Net-(J305-Pad2) renamed /Microcontroller/U1_N
- net Net-(J305-Pad3) renamed /Microcontroller/U1_P
- net Net-(L301-Pad2) renamed /Microcontroller/U2_P
- net Net-(L301-Pad4) renamed /Microcontroller/U2_N
- SW901 pad 1: /FPGA/C0 -> /FPGA/C5
- SW901 pad 2: /FPGA/R0 -> /FPGA/R4
- SW902 pad 1: /FPGA/C1 -> /FPGA/C4
- SW902 pad 2: /FPGA/R0 -> /FPGA/R4
- SW903 pad 1: /FPGA/C2 -> /FPGA/C3
- SW903 pad 2: /FPGA/R0 -> /FPGA/R4
- SW904 pad 1: /FPGA/C3 -> /FPGA/C2
- SW904 pad 2: /FPGA/R0 -> /FPGA/R4
- SW905 pad 1: /FPGA/C4 -> /FPGA/C1
- SW905 pad 2: /FPGA/R0 -> /FPGA/R4
- SW906 pad 1: /FPGA/C5 -> /FPGA/C0
- SW906 pad 2: /FPGA/R0 -> /FPGA/R4
- SW907 pad 1: /FPGA/C0 -> /FPGA/C5
- SW907 pad 2: /FPGA/R1 -> /FPGA/R3
- SW908 pad 1: /FPGA/C1 -> /FPGA/C4
- SW908 pad 2: /FPGA/R1 -> /FPGA/R3
- SW909 pad 1: /FPGA/C2 -> /FPGA/C3
- SW909 pad 2: /FPGA/R1 -> /FPGA/R3
- SW910 pad 1: /FPGA/C3 -> /FPGA/C2
- SW910 pad 2: /FPGA/R1 -> /FPGA/R3
- SW911 pad 1: /FPGA/C4 -> /FPGA/C1
- SW911 pad 2: /FPGA/R1 -> /FPGA/R3
- SW912 pad 1: /FPGA/C5 -> /FPGA/C0
- SW912 pad 2: /FPGA/R1 -> /FPGA/R3
- SW913 pad 1: /FPGA/C0 -> /FPGA/C5
- SW914 pad 1: /FPGA/C1 -> /FPGA/C4
- SW915 pad 1: /FPGA/C2 -> /FPGA/C3
- SW916 pad 1: /FPGA/C3 -> /FPGA/C2
- SW917 pad 1: /FPGA/C4 -> /FPGA/C1
- SW918 pad 1: /FPGA/C5 -> /FPGA/C0
- SW919 pad 1: /FPGA/C0 -> /FPGA/C5
- SW919 pad 2: /FPGA/R3 -> /FPGA/R1
- SW920 pad 1: /FPGA/C1 -> /FPGA/C4
- SW920 pad 2: /FPGA/R3 -> /FPGA/R1
- SW921 pad 1: /FPGA/C2 -> /FPGA/C3
- SW921 pad 2: /FPGA/R3 -> /FPGA/R1
- SW922 pad 1: /FPGA/C3 -> /FPGA/C2
- SW922 pad 2: /FPGA/R3 -> /FPGA/R1
- SW923 pad 1: /FPGA/C4 -> /FPGA/C1
- SW923 pad 2: /FPGA/R3 -> /FPGA/R1
- SW924 pad 1: /FPGA/C5 -> /FPGA/C0
- SW924 pad 2: /FPGA/R3 -> /FPGA/R1
- SW925 pad 1: /FPGA/C0 -> /FPGA/C5
- SW925 pad 2: /FPGA/R4 -> /FPGA/R0
- SW926 pad 1: /FPGA/C1 -> /FPGA/C4
- SW926 pad 2: /FPGA/R4 -> /FPGA/R0
- SW927 pad 1: /FPGA/C2 -> /FPGA/C3
- SW927 pad 2: /FPGA/R4 -> /FPGA/R0
- SW928 pad 1: /FPGA/C3 -> /FPGA/C2
- SW928 pad 2: /FPGA/R4 -> /FPGA/R0
- SW929 pad 1: /FPGA/C4 -> /FPGA/C1
- SW929 pad 2: /FPGA/R4 -> /FPGA/R0
- SW930 pad 1: /FPGA/C5 -> /FPGA/C0
- SW930 pad 2: /FPGA/R4 -> /FPGA/R0
- U1001 pad 89: /Bus Expansion/OPT2_~cs -> /Bus Expansion/6502_OPT2_~cs
- U1001 pad 90: /Bus Expansion/OPT1_~cs -> /Bus Expansion/6502_OPT1_~cs
- U1101 pad 6: /FPGA/RAM_~cs -> /FPGA/6502_RAM_~cs
- U1201 pad 15: /6502/R~W -> /6502/PHI2
- U1201 pad 16: /6502/SYNC -> /6502/PHI1
- U1201 pad 17: /6502/PHI2 -> /6502/SYNC
- U1201 pad 18: /6502/PHI1 -> /6502/R~W
- U1201 pad 2: /6502/6502_PHI1 -> /6502/6502_R~W
- U1201 pad 3: /6502/6502_PHI2 -> /6502/6502_SYNC
- U1201 pad 4: /6502/6502_SYNC -> /6502/6502_PHI1
- U1201 pad 5: /6502/6502_R~W -> /6502/6502_PHI2
- U1205 pad 11: /6502/D7 -> /6502/D0
- U1205 pad 12: /6502/D6 -> /6502/D1
- U1205 pad 13: /6502/D5 -> /6502/D2
- U1205 pad 14: /6502/D4 -> /6502/D3
- U1205 pad 15: /6502/D3 -> /6502/D4
- U1205 pad 16: /6502/D2 -> /6502/D5
- U1205 pad 17: /6502/D1 -> /6502/D6
- U1205 pad 18: /6502/D0 -> /6502/D7
- U1205 pad 2: /6502/B_D0 -> /6502/B_D7
- U1205 pad 3: /6502/B_D1 -> /6502/B_D6
- U1205 pad 4: /6502/B_D2 -> /6502/B_D5
- U1205 pad 5: /6502/B_D3 -> /6502/B_D4
- U1205 pad 6: /6502/B_D4 -> /6502/B_D3
- U1205 pad 7: /6502/B_D5 -> /6502/B_D2
- U1205 pad 8: /6502/B_D6 -> /6502/B_D1
- U1205 pad 9: /6502/B_D7 -> /6502/B_D0
- U1402 pad 14: /FPGA/Physical6502_~BusEnable -> /FPGA/Phys6502_~BusEnable
- U1402 pad 17: /6502/6502_~RES -> /FPGA/Phys6502_~RES
- U1405 pad 15: /FPGA/LED_~CLR -> /FPGA/LED_CLK
- U1405 pad 16: /FPGA/LED_LOAD -> /FPGA/LED_~CLR
- U1405 pad 17: /Display/Din -> /FPGA/LED_DATA
- U1405 pad 18: /Display/CLK -> /FPGA/LED_LOAD
- U1405 pad 19: /Bus Expansion/OPT2_~cs -> /FPGA/OPT2_~cs
- U1405 pad 20: /Bus Expansion/OPT1_~cs -> /FPGA/OPT1_~cs
- U1405 pad 3: /FPGA/RAM_~cs -> /FPGA/6502_RAM_~cs
- U1405 pad 4: /Bus Expansion/OPT1_~cs -> /Bus Expansion/6502_OPT1_~cs
- U1405 pad 5: /Bus Expansion/OPT2_~cs -> /Bus Expansion/6502_OPT2_~cs
- U1405 pad 6: /Display/CLK -> /FPGA/LEDDisp_LOAD
- U1405 pad 8: /FPGA/LED_LOAD -> /FPGA/LEDDisp_~CLR
- U1405 pad 9: /FPGA/LED_~CLR -> /Display/CLK
- U205 pad 112: /FPGA/Physical6502_~BusEnable -> /FPGA/RAM_~cs
- U205 pad 113: /FPGA/RAM_~cs -> /FPGA/OPT1_~cs
- U205 pad 118: /Bus Expansion/OPT1_~cs -> /FPGA/OPT2_~cs
- U205 pad 119: /Bus Expansion/OPT2_~cs -> /FPGA/LED_LOAD
- U205 pad 122: /FPGA/LED_LOAD -> /FPGA/LED_DATA
- U205 pad 123: /Display/Din -> /FPGA/R~W
- U205 pad 124: /Display/CLK -> /FPGA/LED_CLK
- U205 pad 127: /FPGA/PHI2 -> /FPGA/PHI1
- U205 pad 128: /FPGA/PHI1 -> /FPGA/PHI2
- U205 pad 129: /FPGA/R~W -> /FPGA/SYNC
- U205 pad 130: /FPGA/SYNC -> /FPGA/IRQ
- U205 pad 131: /FPGA/IRQ -> /FPGA/RDY
- U205 pad 132: /FPGA/RDY -> /FPGA/~NMI
- U205 pad 135: /FPGA/~NMI -> /FPGA/Phys6502_~RES
- U205 pad 137: /6502/6502_~RES -> /FPGA/RES
- U205 pad 140: /FPGA/RES -> /FPGA/SO
- U205 pad 141: /FPGA/SO -> /FPGA/Phys6502_~BusEnable
- U205 pad 40: /FPGA/G7 -> /FPGA/G0
- U205 pad 41: /FPGA/G6 -> /FPGA/G1
- U205 pad 44: /FPGA/G5 -> /FPGA/G2
- U205 pad 46: /FPGA/G4 -> /FPGA/G3
- U205 pad 47: /FPGA/G3 -> /FPGA/G4
- U205 pad 50: /FPGA/G2 -> /FPGA/G5
- U205 pad 51: /FPGA/G1 -> /FPGA/G6
- U205 pad 52: /FPGA/G0 -> /FPGA/G7
- U205 pad 84: /FPGA/A19 -> /FPGA/A16
- U205 pad 85: /FPGA/A18 -> /FPGA/A17
- U205 pad 86: /FPGA/A17 -> /FPGA/A18
- U205 pad 87: /FPGA/A16 -> /FPGA/A19
- U601 pad 10: /FPGA/LED_LOAD -> /FPGA/LEDDisp_LOAD
- U601 pad 7: /FPGA/LED_~CLR -> /FPGA/LEDDisp_~CLR
- U602 pad 10: /FPGA/LED_LOAD -> /FPGA/LEDDisp_LOAD
- U602 pad 7: /FPGA/LED_~CLR -> /FPGA/LEDDisp_~CLR
- U603 pad 10: /FPGA/LED_LOAD -> /FPGA/LEDDisp_LOAD
- U603 pad 7: /FPGA/LED_~CLR -> /FPGA/LEDDisp_~CLR
- U701 pad 10: /FPGA/LED_LOAD -> /FPGA/LEDDisp_LOAD
- U701 pad 7: /FPGA/LED_~CLR -> /FPGA/LEDDisp_~CLR
- U702 pad 10: /FPGA/LED_LOAD -> /FPGA/LEDDisp_LOAD
- U702 pad 7: /FPGA/LED_~CLR -> /FPGA/LEDDisp_~CLR
- U703 pad 10: /FPGA/LED_LOAD -> /FPGA/LEDDisp_LOAD
- U703 pad 7: /FPGA/LED_~CLR -> /FPGA/LEDDisp_~CLR
- U801 pad 10: /FPGA/LED_LOAD -> /FPGA/LEDDisp_LOAD
- U801 pad 7: /FPGA/LED_~CLR -> /FPGA/LEDDisp_~CLR
- U802 pad 10: /FPGA/LED_LOAD -> /FPGA/LEDDisp_LOAD
- U802 pad 7: /FPGA/LED_~CLR -> /FPGA/LEDDisp_~CLR
- U803 pad 10: /FPGA/LED_LOAD -> /FPGA/LEDDisp_LOAD
- U803 pad 7: /FPGA/LED_~CLR -> /FPGA/LEDDisp_~CLR
Routing:
- net GND: track 0.00 -> 134.8 mm, vias 0 -> 82
- net /6502/A0: track 0.00 -> 78.6 mm
- net /6502/A1: track 0.00 -> 75.2 mm
- net /6502/A2: track 0.00 -> 71.9 mm
- net /6502/A3: track 0.00 -> 68.5 mm
- net /6502/A4: track 0.00 -> 65.2 mm
- net +5V: track 0.00 -> 64.9 mm, vias 0 -> 34
- net +3V3: track 0.00 -> 62.7 mm, vias 0 -> 32
- net /6502/A5: track 0.00 -> 61.8 mm
- net Net-(C202-Pad2): track 0.00 -> 60.6 mm
- net /6502/A6: track 0.00 -> 58.5 mm
- net /6502/A8: track 0.00 -> 57.2 mm
- net /6502/A7: track 0.00 -> 55.2 mm
- net /6502/A9: track 0.00 -> 53.9 mm
- net /6502/A10: track 0.00 -> 50.6 mm
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- added copper zone on F.Cu, net +3V3
- added copper zone on F.Cu, net +5V
- added copper zone on In2.Cu, net +5V
- added copper zone on F.Cu, net GND
- added copper zone on In1.Cu, net GND
- added copper zone on F.Cu, net Net-(C201-Pad2)
- added copper zone on F.Cu, net Net-(C204-Pad1)
- added copper zone on In2.Cu, net Net-(C204-Pad1)
- added copper zone on F.Cu, net Net-(C206-Pad2)
- added copper zone on F.Cu, net Net-(L201-Pad2)
Other:
- board outline added: 228.6 x 184.1 mm
- net class Default: clearance 0.1778 -> 0.1524
- net class Power added: clearance 0.1524, trace_width 0.25, via_dia 0.8, via_drill 0.4
- rule trace_clearance: 0.1778 -> 0.1524
- rule trace_min: 0.2 -> 0.1524
- board text added: "-"
- board text added: "6502 Status Reg"
- board text added: "A"
- board text added: "BRK"
- board text added: "Carry"
- board text added: "Data"
- board text added: "Decimal"
- board text added: "Halt"
- board text added: "IRQ off"
- board text added: "Input/Addr"
- board text added: "Negative"
- board text added: "PC"
- board text added: "Physical 6502"
- board text added: "Run"
- board text added: "SP"
- board text added: "Self-Test Pass"
- board text added: "Soft-CPU"
- board text added: "X"
- board text added: "Y"
- board text added: "Zero"
- board text added: "oVerflow"

Commit message: Most critical nets routed
Parts:
- C1101, C1201, C1202, C1203, C1204, C1205, C1206, C1401, C1402, C1403, C1404, C1405, C1406, C1407, C1408, C1409, C1410, C1411, C1412, C1413, C1414, C1501, C214, C215, C216, C217, C401, C702, Q1301, Q1401, Q1402, Q1403, R1201, R1302, R1304, R1305, R1401, R1402, R1403, R1404, R1405, R1406, R1407, R1501, R1502: moved to B.Cu
- moved R1502 277.8 mm to (226.1, 76.2), turned to 180 degrees
- moved U1501 276.3 mm to (223.5, 76.8), turned to 180 degrees
- moved R1501 268.0 mm to (221.0, 77.5), turned to 180 degrees
- moved C1501 268.0 mm to (221.0, 79.4)
- moved Q1301 249.0 mm to (217.8, 87.0)
- moved Q1401 246.3 mm to (248.3, 88.3)
- moved R1302 238.7 mm to (215.4, 89.7), turned to 180 degrees
- moved Q1403 237.1 mm to (240.0, 88.9), turned to 180 degrees
- moved R1305 236.4 mm to (218.4, 89.7), turned to 180 degrees
- moved Q1402 230.5 mm to (247.0, 95.2), turned to 90 degrees
- moved R1304 227.4 mm to (220.3, 87.0), turned to 90 degrees
- moved C1409 218.6 mm to (240.7, 94.6)
- moved R1402 218.3 mm to (248.3, 90.8)
- moved R1301 212.1 mm to (207.0, 104.1)
- moved J304 210.7 mm to (242.6, 78.7)
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Connections:
- U1001 pad 25: /6502/B_D0 -> Net-(U1001-Pad25)
- U1001 pad 26: /6502/B_D1 -> Net-(U1001-Pad26)
- U1001 pad 27: /6502/B_D2 -> Net-(U1001-Pad27)
- U1001 pad 28: /6502/B_D3 -> Net-(U1001-Pad28)
- U1001 pad 29: /6502/B_D4 -> Net-(U1001-Pad29)
- U1001 pad 30: /6502/B_D5 -> Net-(U1001-Pad30)
- U1001 pad 31: /6502/B_D6 -> Net-(U1001-Pad31)
- U1001 pad 32: /6502/B_D7 -> Net-(U1001-Pad32)
- U1001 pad 45: Net-(U1001-Pad45) -> /6502/B_D0
- U1001 pad 46: Net-(U1001-Pad46) -> /6502/B_D1
- U1001 pad 47: Net-(U1001-Pad47) -> /6502/B_D2
- U1001 pad 48: Net-(U1001-Pad48) -> /6502/B_D3
- U1001 pad 49: Net-(U1001-Pad49) -> /6502/B_D4
- U1001 pad 50: Net-(U1001-Pad50) -> /6502/B_D5
- U1001 pad 51: Net-(U1001-Pad51) -> /6502/B_D6
- U1001 pad 52: Net-(U1001-Pad52) -> /6502/B_D7
- U1001 pad 73: Net-(U1001-Pad73) -> /6502/6502_R~W
- U1001 pad 74: Net-(U1001-Pad74) -> /6502/6502_RDY
- U1001 pad 75: Net-(U1001-Pad75) -> /6502/6502_PHI1
- U1001 pad 76: Net-(U1001-Pad76) -> /6502/6502_PHI0
- U1001 pad 77: Net-(U1001-Pad77) -> /Bus Expansion/6502_OPT2_~cs
- U1001 pad 78: Net-(U1001-Pad78) -> /Bus Expansion/6502_OPT1_~cs
- U1001 pad 79: Net-(U1001-Pad79) -> /6502/6502_SYNC
- U1001 pad 80: Net-(U1001-Pad80) -> /6502/6502_SO
- U1001 pad 81: /6502/6502_R~W -> /Bus Expansion/6502_~RES
- U1001 pad 82: /6502/6502_RDY -> /6502/6502_~NMI
- U1001 pad 83: /6502/6502_PHI1 -> /6502/6502_~IRQ
- U1001 pad 84: /6502/6502_PHI0 -> /6502/6502_PHI2
- U1001 pad 89: /Bus Expansion/6502_OPT2_~cs -> Net-(U1001-Pad89)
- U1001 pad 90: /Bus Expansion/6502_OPT1_~cs -> Net-(U1001-Pad90)
- U1001 pad 91: /6502/6502_SYNC -> Net-(U1001-Pad91)
- U1001 pad 92: /6502/6502_SO -> Net-(U1001-Pad92)
- U1001 pad 93: /Bus Expansion/6502_~RES -> Net-(U1001-Pad93)
- U1001 pad 94: /6502/6502_~NMI -> Net-(U1001-Pad94)
- U1001 pad 95: /6502/6502_~IRQ -> Net-(U1001-Pad95)
- U1001 pad 96: /6502/6502_PHI2 -> Net-(U1001-Pad96)
Routing:
- net GND: track 134.8 -> 286.3 mm, vias 82 -> 184
- net +2V5: track 16.1 -> 142.1 mm, vias 4 -> 27
- net +5V: track 64.9 -> 170.2 mm, vias 34 -> 77
- net +3V3: track 62.7 -> 126.6 mm, vias 32 -> 57
- net +1V2: track 17.0 -> 50.4 mm, vias 4 -> 14
- net /6502/6502_R~W: track 33.1 -> 0.00 mm, vias 2 -> 0
- net /FPGA/Physical6502_~BusEnable: track 29.8 -> 0.00 mm
- net /Microcontroller/USB_N: track 0.00 -> 19.0 mm
- net /Microcontroller/USB_P: track 0.00 -> 18.5 mm
- net Net-(J305-Pad1): track 0.00 -> 6.16 mm
- net Net-(Q1201-Pad3): track 30.2 -> 24.5 mm
- net /Microcontroller/U1_P: track 0.00 -> 5.45 mm
- net /Microcontroller/U2_N: track 0.00 -> 3.33 mm
- net /Microcontroller/U2_P: track 0.00 -> 3.32 mm
- net /Microcontroller/U1_N: track 0.00 -> 3.30 mm
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- added copper zone on F.Cu, net +1V2
- added copper zone on In2.Cu, net +1V2
- added copper zone on B.Cu, net +2V5
- added copper zone on F.Cu, net +2V5
- added copper zone on In2.Cu, net +2V5
- added copper zone on In2.Cu, net +3V3

Commit message: Ready for autorouting
Routing:
- net +5V: track 170.2 -> 178.7 mm, vias 77 -> 80
- net GND: track 286.3 -> 287.8 mm, vias 184 -> 185
Changed lines of the file:
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@@
     (thickness 1.6)
     (drawings 44)
-    (tracks 1878)
+    (tracks 1894)
     (zones 0)
     (modules 337)
@@
   (gr_line (start 167.55971 138.48424) (end 167.55971 140.77024) (layer F.SilkS) (width 0.2))
   (gr_line (start 167.55971 140.77024) (end 167.81371 140.77024) (layer F.SilkS) (width 0.2))
+  (segment (start 253.873 93.345) (end 254 93.472) (width 0.25) (layer F.Cu) (net 6))
+  (via (at 254 93.472) (size 0.8) (drill 0.4) (layers F.Cu B.Cu) (net 6))
+  (segment (start 252.57 93.345) (end 253.873 93.345) (width 0.25) (layer F.Cu) (net 6))
   (segment (start 220.095 120.975) (end 220.745 120.975) (width 0.25) (layer F.Cu) (net 6))
   (segment (start 219.445 120.975) (end 220.095 120.975) (width 0.25) (layer F.Cu) (net 6))
@@
   (segment (start 228.995 102.235) (end 228.727 102.235) (width 0.25) (layer B.Cu) (net 6))
   (via (at 227.584 103.378) (size 0.8) (drill 0.4) (layers F.Cu B.Cu) (net 6))
+  (segment (start 251.46 127) (end 251.935 127) (width 0.25) (layer F.Cu) (net 9))
+  (segment (start 251.935 127) (end 252.57 127.635) (width 0.25) (layer F.Cu) (net 9))
+  (segment (start 252.095 127.635) (end 251.46 127) (width 0.25) (layer B.Cu) (net 9))
+  (segment (start 252.49 127.635) (end 252.095 127.635) (width 0.25) (layer B.Cu) (net 9))
+  (via (at 251.46 127) (size 0.8) (drill 0.4) (layers F.Cu B.Cu) (net 9))
+  (segment (start 265.954 113.3) (end 265.43 112.776) (width 0.25) (layer F.Cu) (net 9))
+  (segment (start 266.7 113.3) (end 265.954 113.3) (width 0.25) (layer F.Cu) (net 9))
+  (via (at 265.43 112.776) (size 0.8) (drill 0.4) (layers F.Cu B.Cu) (net 9))
+  (segment (start 264.16 113.425) (end 266.575 113.425) (width 0.25) (layer F.Cu) (net 9))
+  (segment (start 266.575 113.425) (end 266.7 113.3) (width 0.25) (layer F.Cu) (net 9))
+  (segment (start 210.46624 184.55824) (end 210.312 184.404) (width 0.25) (layer F.Cu) (net 9))
+  (segment (start 212.05121 184.55824) (end 210.46624 184.55824) (width 0.25) (layer F.Cu) (net 9))
+  (via (at 210.312 184.404) (size 0.8) (drill 0.4) (layers F.Cu B.Cu) (net 9))
   (segment (start 173.99 165.255) (end 171.81045 165.255) (width 0.25) (layer B.Cu) (net 9))
   (segment (start 171.81045 165.255) (end 171.67721 165.38824) (width 0.25) (layer B.Cu) (net 9))

Commit message: All nets routed
Routing:
- net /FPGA/R1: track 0.00 -> 295.2 mm, vias 0 -> 1
- net /FPGA/C0: track 0.00 -> 289.7 mm, vias 0 -> 3
- net /FPGA/C3: track 0.00 -> 280.4 mm, vias 0 -> 1
- net /FPGA/R0: track 0.00 -> 277.7 mm, vias 0 -> 3
- net /FPGA/R2: track 0.00 -> 257.2 mm, vias 0 -> 6
- net /FPGA/C1: track 0.00 -> 251.9 mm, vias 0 -> 2
- net /6502/6502_SYNC: track 0.00 -> 228.2 mm, vias 0 -> 3
- net /FPGA/R4: track 0.00 -> 225.5 mm, vias 0 -> 4
- net /FPGA/Physical6502_~BusEnable: track 0.00 -> 225.3 mm, vias 0 -> 4
- net /6502/6502_R~W: track 0.00 -> 222.8 mm, vias 0 -> 5
- net /FPGA/C2: track 0.00 -> 220.0 mm, vias 0 -> 4
- net /FPGA/R3: track 0.00 -> 219.0 mm, vias 0 -> 5
- net /6502/6502_RDY: track 0.00 -> 214.8 mm, vias 0 -> 5
- net /6502/6502_PHI0: track 0.00 -> 213.3 mm, vias 0 -> 2
- net /FPGA/C4: track 0.00 -> 211.6 mm, vias 0 -> 10
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